Commit message: feat: working on eccenters and inertia, urdf

File: urdf/tutorial.urdf (robot description, URDF)
Before this commit: robot microrobot, 7 links, 6 joints
Links:
- added link left_eccenter, mass 10; collision mesh filename=package://microrobot/meshes/test.stl scale=0.05 0.05 0.05; visual mesh filename=package://microrobot/meshes/test.stl scale=0.05 0.05 0.05
- link left_motor: mass None -> ${motor_mass}; geometry collision box size=${motor_depth} ${motor_depth/2} ${motor_depth/2}; visual box size=${motor_depth} ${motor_depth/2} ${motor_depth/2}
- link platform_link: mass None -> ${platform_mass}; geometry collision cylinder length=${platform_thickness} radius=${platform_diameter/2}; visual cylinder length=${platform_thickness} radius=${platform_diameter/2}
- link right_eccenter: mass None -> 10; geometry collision mesh filename=package://microrobot/meshes/test.stl scale=0.05 0.05 0.05; visual mesh filename=package://microrobot/meshes/test.stl scale=0.05 0.05 0.05
- link right_motor: mass None -> ${motor_mass}; geometry collision box size=${motor_depth} ${motor_depth/2} ${motor_depth/2}; visual box size=${motor_depth} ${motor_depth/2} ${motor_depth/2}
- link support_A: mass None -> ${support_mass}; geometry collision sphere radius=${support_diameter}; visual sphere radius=${support_diameter}
- link support_B: mass None -> ${support_mass}; geometry collision sphere radius=${support_diameter}; visual sphere radius=${support_diameter}
- link support_C: mass None -> ${support_mass}; geometry collision sphere radius=${support_diameter}; visual sphere radius=${support_diameter}
Joints:
- added joint left_motor_to_eccenter: type continuous, parent left_motor, child left_eccenter, origin xyz= ${-distance_between_motors/2}                     0                   ${motor_depth/4 + platform_thickness/2}, axis 1 0 0
- joint right_motor_to_eccenter: axis (none) -> 1 0 0; origin (none) -> xyz= ${distance_between_motors/2}                     0                   ${motor_depth/4 + platform_thickness/2}; parent platform_link -> left_motor; type fixed -> continuous
