Commit message: bulk

File: urdf/test.urdf (robot description, URDF)
Before this commit: robot myfirst, 1 links, 0 joints
Links:
- removed link right_tip
- added link base_link
- added link left_eccenter_link, mass 1.825; collision mesh filename=package://microrobot/meshes/large_eccenter_mesh_001.stl; visual mesh filename=package://microrobot/meshes/large_eccenter_mesh_001.stl
- added link platform_link, mass 122; collision mesh filename=package://microrobot/meshes/large_platform_mesh_001.stl; visual mesh filename=package://microrobot/meshes/large_platform_mesh_001.stl
- added link right_eccenter_link, mass 1.825; collision mesh filename=package://microrobot/meshes/large_eccenter_mesh_001.stl; visual mesh filename=package://microrobot/meshes/large_eccenter_mesh_001.stl
Joints:
- added joint platform_joint: type fixed, parent base_link, child platform_link
- added joint platform_to_left_eccenter_joint: type continuous, parent platform_link, child left_eccenter_link, origin xyz=0 0.057 0.008 rpy=0 0 0, axis 0 1 0
- added joint platform_to_right_eccenter_joint: type continuous, parent platform_link, child right_eccenter_link, origin xyz=0 -0.057 0.008 rpy=0 0 -3.14, axis 0 1 0
