Commit message: restart

File: description/microbot.urdf.xacro (robot description, xacro)
@@ -1,4 +1,6 @@
 <?xml version="1.0"?>
 <robot xmlns:xacro="http://www.ros.org/wiki/xacro" name="microrobot">
+    <xacro:include filename="$(find gazebo_ros_motors)/xacro/joint_motor.xacro"/>
     <xacro:include filename="microbot_core.xacro"/>
+    <xacro:include filename="microbot_control.xacro"/>
 </robot>

File: description/microbot_core.xacro (robot description, xacro)
@@ -27,4 +27,5 @@
         <mu1 value="0.4"/>
         <mu2 value="0.4"/>
+        <material>Gazebo/White</material>
     </gazebo>
     <!-- LEFT ECCENTER LINK -->
@@ -34,5 +35,16 @@
         <child link="left_eccenter_link"/>
         <axis xyz="0 1 0"/>
+        <dynamics damping="0.0005" friction="0.0"/>
     </joint>
+    <transmission name="right_motor_transmition">
+    <type>transmission_interface/SimpleTransmission</type>
+        <joint name="platform_to_left_eccenter_joint">
+            <hardwareInterface>EffortJointInterface</hardwareInterface>
+        </joint>
+        <actuator name="r_motor">
+            <hardwareInterface>EffortJointInterface</hardwareInterface>
+            <mechanicalReduction>1</mechanicalReduction>
+        </actuator>
+    </transmission>
     <link name="left_eccenter_link">
         <inertial>
@@ -54,4 +66,7 @@
         </collision>
     </link>
+    <gazebo reference="left_eccenter_link">
+        <material>Gazebo/Blue</material>
+    </gazebo>
     <!-- RIGHT ECCENTER LINK -->
     <joint name="platform_to_right_eccenter_joint" type="continuous">
@@ -60,5 +75,16 @@
         <child link="right_eccenter_link"/>
         <axis xyz="0 1 0"/>
+        <dynamics damping="0.0005" friction="0.0"/>
     </joint>
+    <transmission name="left_motor_transmition">
+    <type>transmission_interface/SimpleTransmission</type>
+        <joint name="platform_to_right_eccenter_joint">
+            <hardwareInterface>EffortJointInterface</hardwareInterface>
+        </joint>
+        <actuator name="l_motor">
+            <hardwareInterface>EffortJointInterface</hardwareInterface>
+            <mechanicalReduction>1</mechanicalReduction>
+        </actuator>
+    </transmission>
     <link name="right_eccenter_link">
         <inertial>
@@ -80,3 +106,6 @@
         </collision>
     </link>
+    <gazebo reference="right_eccenter_link">
+        <material>Gazebo/Blue</material>
+    </gazebo>
 </robot>
