Commit message: add: imu sensor

File: description/microbot.xacro (robot description, xacro)
@@ -111,3 +111,30 @@
         </actuator>
     </transmission>
+    <!--IMU : joint , link , sensor  -->
+    <link name="imu_link">
+        <inertial>
+            <mass value="0.001"/>
+            <origin rpy="0 0 0" xyz="0 0 0"/>
+            <inertia ixx="0.0001" ixy="0" ixz="0" iyy="0.000001" iyz="0" izz="0.0001"/>
+        </inertial>
+        <visual>
+            <origin rpy="0 0 0" xyz="0 0 0"/>
+            <geometry>
+            <box size="0.01 0.01 0.01"/>
+            </geometry>
+            <material name="red"/>
+        </visual>
+        <collision>
+            <origin rpy="0 0 0" xyz="0 0 0"/>
+            <geometry>
+            <box size=".01 .01 .01"/>
+            </geometry>
+        </collision>
+    </link>
+    <joint name="imu_joint" type="fixed">
+        <axis xyz="1 0 0"/>
+        <origin xyz="0 0 0.006"/>
+        <parent link="platform_link"/>
+        <child link="imu_link"/>
+    </joint>
 </robot>

Commit message: add: top down camera, robot_localization working

File: description/microbot.xacro (robot description, xacro)
@@ -13,4 +13,5 @@
         <origin xyz="0 0 -0.002" rpy="0 0 0" />
     </xacro:property>
+    <xacro:property name="camera_link_size" value="0.05" />
     <!-- Base Link -->
     <link name="base_link">
@@ -123,5 +124,4 @@
             <box size="0.01 0.01 0.01"/>
             </geometry>
-            <material name="red"/>
         </visual>
         <collision>
