Commit message: add: platform visual

File: description/actual_robot.xacro (robot description, xacro)
@@ -4,14 +4,25 @@
     <xacro:include filename="actual_microbot.gazebo" />
     <!-- Robot Constants -->
-    <xacro:property name="damping" value="0.000000001" />
+    <xacro:property name="motor_damping" value="0.000000001" />
+    <xacro:property name="platform_height" value="0.0008" />
     <xacro:property name="left_eccenter_position">
-        <origin xyz="0 0.022 0.0042" rpy="0 0 0" />
+        <origin xyz="0 0.022 0.003" rpy="0 0 0" />
     </xacro:property>
     <xacro:property name="right_eccenter_position">
-        <origin xyz="0 -0.022 0.0042" rpy="0 0 -3.14" />
+        <origin xyz="0 -0.022 0.003" rpy="0 0 -3.14" />
     </xacro:property>
-    <xacro:property name="mesh_offset">
+    <xacro:property name="mesh_mass_center_offset">
         <origin xyz="0 0.0015 -0.001" rpy="0 0 0" />
     </xacro:property>
+    <!-- Inertial Macros -->
+    <xacro:macro name="inertial_box" params="mass x y z *origin">
+        <inertial>
+            <xacro:insert_block name="origin"/>
+            <mass value="${mass}" />
+            <inertia ixx="${(1/12) * mass * (y*y+z*z)}" ixy="0.0" ixz="0.0"
+                    iyy="${(1/12) * mass * (x*x+z*z)}" iyz="0.0"
+                    izz="${(1/12) * mass * (x*x+y*y)}" />
+        </inertial>
+    </xacro:macro>
     <!-- Base Link -->
     <link name="base_link">
@@ -24,16 +35,16 @@
     <link name="platform_link">
         <inertial>
-            <mass value="0.018563072"/>
-            <inertia ixx="0.000003360"  ixy="0"  ixz="0" iyy="0.000002453"
-                iyz="0" izz="0.000005762" />
+            <mass value="0.012348768"/>
+            <inertia ixx="0.000002377"  ixy="0"  ixz="0" iyy="0.000001470"
+                iyz="0" izz="0.000003808" />
         </inertial>
         <visual>
             <geometry>
-                <mesh scale="0.001 0.001 0.001" filename="package://microrobot/meshes/microbot_platform_5d.stl"/>
+                <mesh scale="0.001 0.001 0.001" filename="package://microrobot/meshes/ar_platform.dae"/>
             </geometry>
         </visual>
         <collision>
             <geometry>
-                <mesh scale="0.001 0.001 0.001" filename="package://microrobot/meshes/microbot_platform_5d.stl"/>
+                <mesh scale="0.001 0.001 0.001" filename="package://microrobot/meshes/platform collision mesh v7.stl"/>
             </geometry>
         </collision>
@@ -42,5 +53,5 @@
     <link name="left_eccenter_link">
         <inertial>
-            <xacro:insert_block name="mesh_offset" />
+            <xacro:insert_block name="mesh_mass_center_offset" />
             <mass value="0.000147969"/>
             <inertia ixx="1.523e-10"  ixy="0"  ixz="0" iyy="1.893e-10" iyz="0" izz="2.589e-10" />
@@ -62,10 +73,10 @@
         <child link="left_eccenter_link"/>
         <axis xyz="0 1 0"/>
-        <dynamics damping="${damping}" friction="0.0"/>
+        <dynamics damping="${motor_damping}" friction="0.0"/>
     </joint>
     <!-- Right eccenter link -->
     <link name="right_eccenter_link">
         <inertial>
-            <xacro:insert_block name="mesh_offset" />
+            <xacro:insert_block name="mesh_mass_center_offset" />
             <mass value="0.000147969"/>
             <inertia ixx="1.523e-10"  ixy="0"  ixz="0" iyy="1.893e-10" iyz="0" izz="2.589e-10" />
@@ -87,5 +98,50 @@
         <child link="right_eccenter_link"/>
         <axis xyz="0 1 0"/>
-        <dynamics damping="${damping}" friction="0.0"/>
+        <dynamics damping="${motor_damping}" friction="0.0"/>
     </joint>
+    <!-- IMU link -->
+    <link name="imu_link">
+        <xacro:inertial_box mass="0.00001" x="0.001" y="0.001" z="0.001">
+            <origin xyz="0.0005 0 0.0005" rpy="0 0 0"/>
+        </xacro:inertial_box>
+        <visual>
+            <origin rpy="0 0 0" xyz="0 0 0"/>
+            <geometry>
+            <box size="0.001 0.001 0.001"/>
+            </geometry>
+        </visual>
+        <collision>
+            <origin rpy="0 0 0" xyz="0 0 0"/>
+            <geometry>
+            <box size="0.001 0.001 0.001"/>
+            </geometry>
+        </collision>
+    </link>
+    <joint name="imu_joint" type="fixed">
+        <axis xyz="1 0 0"/>
+        <origin xyz="0 0 ${platform_height + 0.0005}"/>
+        <parent link="platform_link"/>
+        <child link="imu_link"/>
+    </joint>
+    <!-- Transmitions -->
+        <transmission name="left_motor_transmition">
+        <type>transmission_interface/SimpleTransmission</type>
+        <joint name="platform_to_left_eccenter_joint">
+            <hardwareInterface>hardware_interface/VelocityJointInterface </hardwareInterface>
+        </joint>
+        <actuator name="l_motor">
+            <hardwareInterface>hardware_interface/VelocityJointInterface </hardwareInterface>
+            <mechanicalReduction>1</mechanicalReduction>
+        </actuator>
+    </transmission>
+	<transmission name="right_motor_transmition">
+        <type>transmission_interface/SimpleTransmission</type>
+        <joint name="platform_to_right_eccenter_joint">
+            <hardwareInterface>hardware_interface/VelocityJointInterface </hardwareInterface>
+        </joint>
+        <actuator name="r_motor">
+            <hardwareInterface>hardware_interface/VelocityJointInterface </hardwareInterface>
+            <mechanicalReduction>1</mechanicalReduction>
+        </actuator>
+    </transmission>
 </robot>

File: description/camera.xacro (robot description, xacro)
@@ -5,5 +5,5 @@
     <link name="camera base"></link>
     <joint name="my_joint" type="fixed">
-        <origin xyz="0 0 1" rpy="0 1.57 0"/>
+        <origin xyz="0 0 0.15" rpy="0 1.57 0"/>
         <parent link="camera base"/>
         <child link="camera_link"/>
@@ -41,6 +41,6 @@
             </image>
             <clip>
-            <near>0.1</near>
-            <far>100</far>
+            <near>0.001</near>
+            <far>10</far>
             </clip>
             <noise>

Commit message: add: ar tag

File: description/actual_robot.xacro (robot description, xacro)
@@ -41,5 +41,5 @@
         <visual>
             <geometry>
-                <mesh scale="0.001 0.001 0.001" filename="package://microrobot/meshes/ar_platform.dae"/>
+                <mesh scale="0.001 0.001 0.001" filename="package://microrobot/meshes/platform visual v2.stl"/>
             </geometry>
         </visual>
@@ -108,5 +108,5 @@
             <origin rpy="0 0 0" xyz="0 0 0"/>
             <geometry>
-            <box size="0.001 0.001 0.001"/>
+                <box size="0.001 0.001 0.001"/>
             </geometry>
         </visual>
@@ -124,6 +124,30 @@
         <child link="imu_link"/>
     </joint>
+    <!-- AR tag -->
+    <link name="ar_tag_link">
+        <xacro:inertial_box mass="0.00001" x="0.03" y="0.03" z="0.005">
+            <origin xyz="0.0005 0 0.0005" rpy="0 0 0"/>
+        </xacro:inertial_box>
+        <visual>
+            <origin rpy="0 0 0" xyz="0 0 0"/>
+            <geometry>
+                <mesh filename="package://microrobot/meshes/ar_tag_3cm.dae"/>
+            </geometry>
+        </visual>
+        <collision>
+            <origin rpy="0 0 0" xyz="0 0 0"/>
+            <geometry>
+                <mesh filename="package://microrobot/meshes/ar_tag_3cm.dae"/>
+            </geometry>
+        </collision>
+    </link>
+    <joint name="ar_tag_joint" type="fixed">
+        <axis xyz="1 0 0"/>
+        <origin xyz="0 0 0.014"/>
+        <parent link="platform_link"/>
+        <child link="ar_tag_link"/>
+    </joint>
     <!-- Transmitions -->
-        <transmission name="left_motor_transmition">
+    <transmission name="left_motor_transmition">
         <type>transmission_interface/SimpleTransmission</type>
         <joint name="platform_to_left_eccenter_joint">

Commit message: fix: velocity controllers error, naming

File: description/actual_robot.xacro (robot description, xacro)
@@ -4,11 +4,12 @@
     <xacro:include filename="actual_microbot.gazebo" />
     <!-- Robot Constants -->
-    <xacro:property name="motor_damping" value="0.000000001" />
+    <xacro:property name="motor_damping" value="0.00000000" />
+    <xacro:property name="motor_friction" value="0.00000" />
     <xacro:property name="platform_height" value="0.0008" />
     <xacro:property name="left_eccenter_position">
-        <origin xyz="0 0.022 0.003" rpy="0 0 0" />
+        <origin xyz="0 0.022 0.0032" rpy="0 0 0" />
     </xacro:property>
     <xacro:property name="right_eccenter_position">
-        <origin xyz="0 -0.022 0.003" rpy="0 0 -3.14" />
+        <origin xyz="0 -0.022 0.0032" rpy="0 0 -3.14" />
     </xacro:property>
     <xacro:property name="mesh_mass_center_offset">
@@ -35,11 +36,11 @@
     <link name="platform_link">
         <inertial>
-            <mass value="0.012348768"/>
-            <inertia ixx="0.000002377"  ixy="0"  ixz="0" iyy="0.000001470"
-                iyz="0" izz="0.000003808" />
+            <mass value="0.100003017"/>
+            <inertia ixx="0.000019251"  ixy="0"  ixz="0" iyy="0.000011903"
+                iyz="0" izz="0.000030834" />
         </inertial>
         <visual>
             <geometry>
-                <mesh scale="0.001 0.001 0.001" filename="package://microrobot/meshes/platform visual v2.stl"/>
+                <mesh scale="0.001 0.001 0.001" filename="package://microrobot/meshes/platform collision mesh v7.stl"/>
             </geometry>
         </visual>
@@ -54,6 +55,6 @@
         <inertial>
             <xacro:insert_block name="mesh_mass_center_offset" />
-            <mass value="0.000147969"/>
-            <inertia ixx="1.523e-10"  ixy="0"  ixz="0" iyy="1.893e-10" iyz="0" izz="2.589e-10" />
+            <mass value="0.000208337"/>
+            <inertia ixx="2.145e-10"  ixy="0"  ixz="0" iyy="2.666e-10" iyz="0" izz="3.646e-10" />
         </inertial>
         <visual>
@@ -73,5 +74,5 @@
         <child link="left_eccenter_link"/>
         <axis xyz="0 1 0"/>
-        <dynamics damping="${motor_damping}" friction="0.0"/>
+        <dynamics damping="${motor_damping}" friction="${motor_friction}"/>
     </joint>
     <!-- Right eccenter link -->
@@ -79,6 +80,6 @@
         <inertial>
             <xacro:insert_block name="mesh_mass_center_offset" />
-            <mass value="0.000147969"/>
-            <inertia ixx="1.523e-10"  ixy="0"  ixz="0" iyy="1.893e-10" iyz="0" izz="2.589e-10" />
+            <mass value="0.000208337"/>
+            <inertia ixx="2.145e-10"  ixy="0"  ixz="0" iyy="2.666e-10" iyz="0" izz="3.646e-10" />
         </inertial>
         <visual>
@@ -98,5 +99,5 @@
         <child link="right_eccenter_link"/>
         <axis xyz="0 1 0"/>
-        <dynamics damping="${motor_damping}" friction="0.0"/>
+        <dynamics damping="${motor_damping}" friction="${motor_friction}"/>
     </joint>
     <!-- IMU link -->

File: description/camera.xacro (robot description, xacro)
@@ -56,5 +56,5 @@
             <alwaysOn>true</alwaysOn>
             <updateRate>0.0</updateRate>
-            <cameraName>rrbot/camera1</cameraName>
+            <cameraName>microbot/camera1</cameraName>
             <imageTopicName>image_raw</imageTopicName>
             <cameraInfoTopicName>camera_info</cameraInfoTopicName>

Commit message: add: fixed ar tag detection

File: description/actual_robot.xacro (robot description, xacro)
@@ -8,8 +8,8 @@
     <xacro:property name="platform_height" value="0.0008" />
     <xacro:property name="left_eccenter_position">
-        <origin xyz="0 0.022 0.0032" rpy="0 0 0" />
+        <origin xyz="0 0.022 0.003" rpy="0 0 0" />
     </xacro:property>
     <xacro:property name="right_eccenter_position">
-        <origin xyz="0 -0.022 0.0032" rpy="0 0 -3.14" />
+        <origin xyz="0 -0.022 0.003" rpy="0 0 -3.14" />
     </xacro:property>
     <xacro:property name="mesh_mass_center_offset">
@@ -127,5 +127,5 @@
     <!-- AR tag -->
     <link name="ar_tag_link">
-        <xacro:inertial_box mass="0.00001" x="0.03" y="0.03" z="0.005">
+        <xacro:inertial_box mass="0.00001" x="0.03" y="0.03" z="0.001">
             <origin xyz="0.0005 0 0.0005" rpy="0 0 0"/>
         </xacro:inertial_box>
@@ -133,5 +133,5 @@
             <origin rpy="0 0 0" xyz="0 0 0"/>
             <geometry>
-                <mesh filename="package://microrobot/meshes/ar_tag_3cm.dae"/>
+                <mesh filename="package://microrobot/ar_tags/ar_tag_0_3cm.dae"/>
             </geometry>
         </visual>
@@ -139,5 +139,5 @@
             <origin rpy="0 0 0" xyz="0 0 0"/>
             <geometry>
-                <mesh filename="package://microrobot/meshes/ar_tag_3cm.dae"/>
+                <mesh filename="package://microrobot/ar_tags/ar_tag_0_3cm.dae"/>
             </geometry>
         </collision>

File: description/camera.xacro (robot description, xacro)
@@ -34,5 +34,5 @@
         <update_rate>30.0</update_rate>
         <camera name="head">
-            <horizontal_fov>1.047</horizontal_fov>
+            <horizontal_fov>1</horizontal_fov>
             <image>
             <width>800</width>
@@ -43,12 +43,12 @@
             <near>0.001</near>
             <far>10</far>
-            </clip>
+            </clip>SA
             <noise>
-            <type>gaussian</type>
-            <!-- Noise is sampled independently per pixel on each frame.
-                That pixel's noise value is added to each of its color
-                channels, which at that point lie in the range [0,1]. -->
-            <mean>0.0</mean>
-            <stddev>0.007</stddev>
+                <type>gaussian</type>
+                <!-- Noise is sampled independently per pixel on each frame.
+                    That pixel's noise value is added to each of its color
+                    channels, which at that point lie in the range [0,1]. -->
+                <mean>0.0</mean>
+                <stddev>0.0</stddev>
             </noise>
         </camera>

Commit message: add: visual odometry publisher

File: description/actual_robot.xacro (robot description, xacro)
@@ -42,5 +42,5 @@
         <visual>
             <geometry>
-                <mesh scale="0.001 0.001 0.001" filename="package://microrobot/meshes/platform collision mesh v7.stl"/>
+                <mesh scale="0.001 0.001 0.001" filename="package://microrobot/meshes/platform visual v2.stl"/>
             </geometry>
         </visual>
@@ -131,5 +131,5 @@
         </xacro:inertial_box>
         <visual>
-            <origin rpy="0 0 0" xyz="0 0 0"/>
+            <origin rpy="0 0 1.57079633" xyz="0 0 0"/>
             <geometry>
                 <mesh filename="package://microrobot/ar_tags/ar_tag_0_3cm.dae"/>

File: description/camera.xacro (robot description, xacro)
@@ -5,5 +5,5 @@
     <link name="camera base"></link>
     <joint name="my_joint" type="fixed">
-        <origin xyz="0 0 0.15" rpy="0 1.57 0"/>
+        <origin xyz="0 0 0.15" rpy="0 1.57 -1.57"/>
         <parent link="camera base"/>
         <child link="camera_link"/>

Commit message: add: restarted low level controller

File: description/actual_robot.xacro (robot description, xacro)
@@ -5,6 +5,6 @@
     <!-- Robot Constants -->
     <!-- TODO: damping and friction may limit jitter -->
-    <xacro:property name="motor_damping" value="0.00000000" />
-    <xacro:property name="motor_friction" value="0.00000" />
+    <xacro:property name="motor_damping" value="1e-7" /> <!-- highest damping possible 0.000001-->
+    <xacro:property name="motor_friction" value="0.0" />
     <xacro:property name="platform_height" value="0.0008" />
     <xacro:property name="left_eccenter_position">
@@ -27,4 +27,13 @@
         </inertial>
     </xacro:macro>
+     <xacro:macro name="inertial_cylinder" params="mass length radius *origin">
+        <inertial>
+            <xacro:insert_block name="origin"/>
+            <mass value="${mass}" />
+            <inertia ixx="${(1/12) * mass * (3*radius*radius + length*length)}" ixy="0.0" ixz="0.0"
+                    iyy="${(1/12) * mass * (3*radius*radius + length*length)}" iyz="0.0"
+                    izz="${(1/2) * mass * (radius*radius)}" />
+        </inertial>
+    </xacro:macro>
     <!-- Base Link -->
     <link name="base_link">
@@ -41,12 +50,18 @@
                 iyz="0" izz="0.000030834" />
         </inertial>
+        <!-- <xacro:inertial_cylinder mass="0.1" length="0.0006" radius="0.05">
+            <origin xyz="0 0 0" rpy="0 0 0"/>
+        </xacro:inertial_cylinder>
+         -->
         <visual>
             <geometry>
-                <mesh scale="0.001 0.001 0.001" filename="package://microrobot/meshes/platform visual v2.stl"/>
+                <mesh scale="0.001 0.001 0.001"
+                    filename="package://microrobot/meshes/platform visual v2.stl"/>
             </geometry>
         </visual>
         <collision>
             <geometry>
-                <mesh scale="0.001 0.001 0.001" filename="package://microrobot/meshes/platform collision mesh v7.stl"/>
+                <mesh scale="0.001 0.001 0.001"
+                    filename="package://microrobot/meshes/platform collision mesh v7.stl"/>
             </geometry>
         </collision>
@@ -57,14 +72,17 @@
             <xacro:insert_block name="mesh_mass_center_offset" />
             <mass value="0.000208337"/>
-            <inertia ixx="2.145e-10"  ixy="0"  ixz="0" iyy="2.666e-10" iyz="0" izz="3.646e-10" />
+            <inertia ixx="2.145e-10"  ixy="0"  ixz="0" iyy="2.666e-10" iyz="0"
+                izz="3.646e-10" />
         </inertial>
         <visual>
             <geometry>
-                <mesh scale="0.001 0.001 0.001" filename="package://microrobot/meshes/microbot_eccenter_5d.stl"/>
+                <mesh scale="0.001 0.001 0.001"
+                    filename="package://microrobot/meshes/microbot_eccenter_5d.stl"/>
             </geometry>
         </visual>
         <collision>
             <geometry>
-                <mesh scale="0.001 0.001 0.001" filename="package://microrobot/meshes/microbot_eccenter_5d.stl"/>
+                <mesh scale="0.001 0.001 0.001"
+                    filename="package://microrobot/meshes/microbot_eccenter_5d.stl"/>
             </geometry>
         </collision>
@@ -82,14 +100,17 @@
             <xacro:insert_block name="mesh_mass_center_offset" />
             <mass value="0.000208337"/>
-            <inertia ixx="2.145e-10"  ixy="0"  ixz="0" iyy="2.666e-10" iyz="0" izz="3.646e-10" />
+            <inertia ixx="2.145e-10"  ixy="0"  ixz="0" iyy="2.666e-10" iyz="0"
+                izz="3.646e-10" />
         </inertial>
         <visual>
             <geometry>
-                <mesh scale="0.001 0.001 0.001" filename="package://microrobot/meshes/microbot_eccenter_5d.stl"/>
+                <mesh scale="0.001 0.001 0.001"
+                    filename="package://microrobot/meshes/microbot_eccenter_5d.stl"/>
             </geometry>
         </visual>
         <collision>
             <geometry>
-                <mesh scale="0.001 0.001 0.001" filename="package://microrobot/meshes/microbot_eccenter_5d.stl"/>
+                <mesh scale="0.001 0.001 0.001"
+                    filename="package://microrobot/meshes/microbot_eccenter_5d.stl"/>
             </geometry>
         </collision>
@@ -116,5 +137,5 @@
             <origin rpy="0 0 0" xyz="0 0 0"/>
             <geometry>
-            <box size="0.001 0.001 0.001"/>
+                <box size="0.001 0.001 0.001"/>
             </geometry>
         </collision>

File: description/camera.xacro (robot description, xacro)
@@ -25,5 +25,5 @@
             <mass value="1e-5" />
             <origin xyz="0 0 0" rpy="0 0 0"/>
-            <inertia ixx="1e-6" ixy="0" ixz="0" iyy="1e-6" iyz="0" izz="1e-6" />
+            <inertia ixx="1e-9" ixy="0" ixz="0" iyy="1e-9" iyz="0" izz="1e-9" />
         </inertial>
     </link>

Commit message: add: theta orientation controller

File: description/actual_robot.xacro (robot description, xacro)
@@ -5,6 +5,6 @@
     <!-- Robot Constants -->
     <!-- TODO: damping and friction may limit jitter -->
-    <xacro:property name="motor_damping" value="1e-7" /> <!-- highest damping possible 0.000001-->
-    <xacro:property name="motor_friction" value="0.0" />
+    <xacro:property name="motor_damping" value="0.0" />
+    <xacro:property name="motor_friction" value="1e-4" />
     <xacro:property name="platform_height" value="0.0008" />
     <xacro:property name="left_eccenter_position">

Commit message: feat: setup launchfile for multiple robots, re-added ar tag

File: description/actual_robot.xacro (robot description, xacro)
@@ -151,5 +151,5 @@
     </joint> -->
     <!-- AR tag -->
-    <!-- <link name="ar_tag_link">
+    <link name="ar_tag_link">
         <xacro:inertial_box mass="0.00001" x="0.03" y="0.03" z="0.001">
             <origin xyz="0.0005 0 0.0005" rpy="0 0 0"/>
@@ -173,5 +173,5 @@
         <parent link="platform_link"/>
         <child link="ar_tag_link"/>
-    </joint> -->
+    </joint>
     <!-- Transmitions -->
     <!-- <transmission name="left_motor_transmition">

Commit message: physics testing

File: description/actual_robot.xacro (robot description, xacro)
@@ -127,5 +127,5 @@
     </joint>
     <!-- IMU link -->
-    <!-- <link name="imu_link">
+    <link name="imu_link">
         <xacro:inertial_box mass="0.00001" x="0.001" y="0.001" z="0.001">
             <origin xyz="0.0005 0 0.0005" rpy="0 0 0"/>
@@ -149,5 +149,5 @@
         <parent link="platform_link"/>
         <child link="imu_link"/>
-    </joint> -->
+    </joint>
     <!-- AR tag -->
     <link name="ar_tag_link">

Commit message: fix: all tf

File: description/actual_robot.xacro (robot description, xacro)
@@ -1,4 +1,4 @@
 <?xml version="1.0"?>
-<robot name="microrobot" xmlns:xacro="http://www.ros.org/wiki/xacro" >
+<robot name="microbot" xmlns:xacro="http://www.ros.org/wiki/xacro" >
     <!-- Import all Gazebo-customization elements, including Gazebo colors -->
     <xacro:include filename="actual_microbot.gazebo" />
@@ -57,5 +57,5 @@
             <geometry>
                 <mesh scale="0.001 0.001 0.001"
-                    filename="package://microrobot/meshes/platform collision mesh v7.stl"/>
+                    filename="package://microrobot/meshes/platform visual v2.stl"/>
             </geometry>
         </visual>
@@ -170,6 +170,6 @@
     <joint name="ar_tag_joint" type="fixed">
         <axis xyz="1 0 0"/>
-        <origin xyz="0 0 0.014"/>
-        <parent link="platform_link"/>
+        <origin xyz="0 0 0.014" rpy="0 0 1.57"/>
+        <parent link="base_link"/>
         <child link="ar_tag_link"/>
     </joint>
