Commit message: more stable movement, trying to minimize bounce

File: description/actual_robot.xacro (robot description, xacro)
@@ -6,5 +6,5 @@
     <!-- TODO: damping and friction may limit jitter -->
     <xacro:property name="motor_damping" value="0.00000001" />
-    <xacro:property name="motor_friction" value="0.0" />
+    <xacro:property name="motor_friction" value="0.00001" />
     <xacro:property name="platform_height" value="0.0008" />
     <xacro:property name="left_eccenter_position">
@@ -65,7 +65,7 @@
                     filename="package://microrobot/meshes/platform collision mesh v7.stl"/>
             </geometry>
-            <surface>
+            <!-- <surface>
                 <bounce restitution_coefficient="0" threshold="0"/>
-            </surface>
+            </surface> -->
         </collision>
     </link>

Commit message: repo clean up

File: description/actual_robot.xacro (robot description, xacro)
@@ -158,5 +158,5 @@
             <origin rpy="0 0 1.57079633" xyz="0 0 0"/>
             <geometry>
-                <mesh filename="package://microrobot/ar_tags/ar_tag_0_3cm.dae"/>
+                <mesh filename="package://microrobot/ar_tags/ar_tag_0/ar_tag_0_3cm.dae"/>
             </geometry>
         </visual>
@@ -164,5 +164,5 @@
             <origin rpy="0 0 0" xyz="0 0 0"/>
             <geometry>
-                <mesh filename="package://microrobot/ar_tags/ar_tag_0_3cm.dae"/>
+                <mesh filename="package://microrobot/ar_tags/ar_tag_0/ar_tag_0_3cm.dae"/>
             </geometry>
         </collision>

Commit message: clothoid fix

File: description/actual_robot.xacro (robot description, xacro)
@@ -4,5 +4,4 @@
     <xacro:include filename="actual_microbot.gazebo" />
     <!-- Robot Constants -->
-    <!-- TODO: damping and friction may limit jitter -->
     <xacro:property name="motor_damping" value="0.00000001" />
     <xacro:property name="motor_friction" value="0.00001" />
@@ -171,5 +170,5 @@
         <axis xyz="1 0 0"/>
         <origin xyz="0 0 0.014" rpy="0 0 1.57"/>
-        <parent link="base_link"/>
+        <parent link="platform_link"/>
         <child link="ar_tag_link"/>
     </joint>
